File: Kicad/Soundalyser.kicad_pcb (KiCad board)
At the start: 2 copper layers, 87.6 x 85.3 mm, 16 parts, among them SW1 RotaryEncoder_Switch, U1 XIAO-RP2040-DIP

Commit message: updated microsd card reader
Parts:
- G***: moved to F.Cu
- moved U4 20.0 mm to (110.2, 89.9)
- moved G*** 15.2 mm to (106.8, 73.1), turned to 0 degrees
- moved G*** 14.8 mm to (111.6, 79.2)
- moved G*** 14.8 mm to (111.4, 74.4)
Connections:
- U4 pad 2: +5V -> +3.3V
Routing:
- net +5V: track 46.8 -> 0.00 mm, vias 3 -> 0
- net GPIO28: track 100.8 -> 126.3 mm, vias 0 -> 1
- net GPIO27: track 121.7 -> 98.0 mm
- net MOSI: track 48.8 -> 28.7 mm, vias 0 -> 1
- net GPIO26: track 83.8 -> 102.3 mm
- net SDA: track 89.6 -> 75.3 mm
- net SCK: track 40.8 -> 26.5 mm
- net GPIO0: track 59.6 -> 46.3 mm, vias 2 -> 1
- net MISO: track 41.5 -> 30.0 mm
- net +3.3V: track 111.2 -> 117.5 mm, vias 0 -> 2
- net SCL: track 81.0 -> 76.9 mm, vias 1 -> 0
- net GND: track 178.1 -> 174.7 mm, vias 3 -> 2
- net GPIO1: track 26.2 -> 24.4 mm, vias 1 -> 0
- net GPIO29: track 84.0 -> 82.7 mm, vias 1 -> 3
